File: ToyaPcb-FIRST HERE/ToyaPcb.kicad_pcb (KiCad board)
At the start: 2 copper layers, 199.9 x 300 mm, 37 parts

Commit message: bug fix
firmware bug fix
PCB dimension fix
Parts:
- added REF**: Buzzer_12x9.5RM7.6, Buzzer_Beeper:Buzzer_12x9.5RM7.6, F.Cu at (148.3, 53.7)
- added REF**: TO-92_Horizontal2, Package_TO_SOT_THT:TO-92_Horizontal2, F.Cu at (153.9, 50.7)
- added REF**: R_Axial_DIN0207_L6.3mm_D2.5mm_P10.16mm_Horizontal, Resistor_THT:R_Axial_DIN0207_L6.3mm_D2.5mm_P10.16mm_Horizontal, F.Cu at (151.2, 47.3)
- added REF**: Buzzer_12x9.5RM7.6, Buzzer_Beeper:Buzzer_12x9.5RM7.6, F.Cu at (22.2, 295.9)
- added REF**: Buzzer_12x9.5RM7.6, Buzzer_Beeper:Buzzer_12x9.5RM7.6, F.Cu at (195.4, 295.9)
- added REF**: R_Axial_DIN0207_L6.3mm_D2.5mm_P10.16mm_Horizontal, Resistor_THT:R_Axial_DIN0207_L6.3mm_D2.5mm_P10.16mm_Horizontal, F.Cu at (154.3, 55.9)
- moved ? 20.2 mm to (76.0, 250.9)
- moved REF** 20.0 mm to (68.2, 106.5)
- moved ? 20.0 mm to (20.9, 194.2)
- moved ? 20.0 mm to (133.4, 253.7)
- moved REF** 20.0 mm to (79.5, 138.2)
- moved REFe 20.0 mm to (169.8, 209.2)
- moved REFe 20.0 mm to (8.33, 206.3)
- moved G*** 20.0 mm to (100.7, 56.4) (x2)
- moved REF** 20.0 mm to (174.4, 58.6)
- moved REF** 20.0 mm to (31.0, 91.2)
- moved REF** 20.0 mm to (72.3, 87.7)
- moved REF** 20.0 mm to (177.3, 38.4)
- moved REF** 20.0 mm to (138.5, 81.5)
- moved REF** 20.0 mm to (195.3, 82.3)
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Connections:
- REF** pad 2: BEBAS -> G (x3)
- REF** pad 1: BEBAS -> G (x5)
- REF** pad 4: BEBAS -> G (x6)
- REF** pad 2: BEBAS -> VCC
- REF** pad 5: BEBAS -> VCC (x2)
- REF** pad 18: data -> BEBAS
- REF** pad 19: BEBAS -> data
- REF** pad 9: BEBAS -> VCC
- REFe pad 1: BEBAS -> G (x9)
- REFe pad 4: BEBAS -> G (x9)
Routing:
- net BEBAS: track 0.00 -> 2836.2 mm, vias 29 -> 2
- net data: track 0.00 -> 1012.9 mm, vias 2 -> 1
- net VCC: track 0.00 -> 988.2 mm
- net G: track 0.00 -> 830.6 mm, vias 1 -> 8
- net (no net): track 0.00 -> 16.5 mm
- net buzzer: track 0.00 -> 4.92 mm
- added copper zone on B.Cu, net G
- added copper zone on F.Cu, net VCC
Other:
- board text added: "REV ENAM"
- board text added: "TR9012 ECB"
- board text removed: "REV TIGA"

Commit message: A lot Of thing changed
i dont even remember what changed LOL
Parts:
- removed the G*** at (100.7, 56.4)
- added ?: , , F.Cu at (186.7, 178.5)
- added ?: , , F.Cu at (102.3, 97.8)
- added ?: , , F.Cu at (39.5, 240.1)
- added ?: , , F.Cu at (102.7, 124.7)
- added ?: , , F.Cu at (34.1, 160.3)
- added ?: , , F.Cu at (100.3, 248.1)
- added ?: , , F.Cu at (202.7, 306.2)
- added ?: , , F.Cu at (4.67, 306.2)
- added ?: , , F.Cu at (202.7, 8.05)
- added REF**: PinHeader_1x02_P2.54mm_Vertical, Connector_PinHeader_2.54mm:PinHeader_1x02_P2.54mm_Vertical, F.Cu at (174.6, 56.5)
- added REF**: PinHeader_1x02_P2.54mm_Vertical, Connector_PinHeader_2.54mm:PinHeader_1x02_P2.54mm_Vertical, F.Cu at (174.4, 60.3)
- added REF**: PinHeader_1x10_P2.54mm_Vertical, Connector_PinHeader_2.54mm:PinHeader_1x10_P2.54mm_Vertical, F.Cu at (174.6, 56.5)
- moved REF** 7.60 mm to (145.1, 46.9)
- moved G*** 7.35 mm to (101.2, 49.1)
- moved REF** 5.30 mm to (151.8, 45.8)
- moved REF** 5.30 mm to (149.1, 42.4)
- moved REF** 5.05 mm to (152.7, 51.2)
- moved REF** 3.96 mm to (7.57, 55.1)
- moved REF** 1.65 mm to (174.4, 60.3)
Routing:
- net VCC: track 988.2 -> 1353.7 mm, vias 0 -> 1
- net G: track 830.6 -> 972.6 mm, vias 8 -> 16
- net BEBAS: track 2836.2 -> 2862.7 mm
- net (no net): track 16.5 -> 19.5 mm
- added copper zone on F.Cu, net G
- removed copper zone on F.Cu, net VCC
Other:
- board text added: "FUN.TOYA"
- board text removed: "REV ENAM"

Commit message: Major changes
simple game removed
improvised simon Say game
custom font for each board (font not yet implemented for other board)
rotated screen to  compensate pcb revision
2 extra PCB file
etc
Parts:
- added REF**: PinHeader_1x03_P2.54mm_Vertical, Connector_PinHeader_2.54mm:PinHeader_1x03_P2.54mm_Vertical, F.Cu at (11.5, 60.9)
- added REF**: PinHeader_1x03_P2.54mm_Vertical, Connector_PinHeader_2.54mm:PinHeader_1x03_P2.54mm_Vertical, F.Cu at (11.5, 56.5)
- moved G*** 16.3 mm to (117.5, 49.4)
- moved REF** 16.2 mm to (21.8, 47.3)
- moved REF** 11.5 mm to (9.80, 25.5)
Routing:
- net BEBAS: track 2862.7 -> 2840.0 mm
- net VCC: track 1353.7 -> 1346.6 mm
- net G: vias 16 -> 17
